File: FRDM-MCXA153_shield_template.kicad_pcb (KiCad board)
At the start: 2 copper layers, 101.4 x 54.6 mm, 10 parts, among them J1 Conn_02x08_Odd_Even, J2 Conn_02x10_Odd_Even, J3 Conn_02x08_Odd_Even, J4 Conn_02x06_Odd_Even, J5 Conn_01x08_Pin, J6 Conn_01x08_Pin

Commit message: add power module
Parts:
- added BT1: Battery_Cell, Connector_Wire:SolderWire-0.75sqmm_1x02_P4.8mm_D1.25mm_OD2.3mm, F.Cu at (119.7, 98.0)
- added BT2: Battery_Cell, Connector_Wire:SolderWire-0.75sqmm_1x02_P4.8mm_D1.25mm_OD2.3mm, F.Cu at (119.7, 93.4)
- added C1: 100n, Capacitor_SMD:C_1206_3216Metric_Pad1.33x1.80mm_HandSolder, F.Cu at (116.9, 88.3)
- added C2: 2.2n, Capacitor_SMD:C_1206_3216Metric_Pad1.33x1.80mm_HandSolder, F.Cu at (110.8, 83.3)
- added C3: 1u, Capacitor_SMD:C_1206_3216Metric_Pad1.33x1.80mm_HandSolder, F.Cu at (127.2, 68.5)
- added C4: 10u, Capacitor_SMD:C_1206_3216Metric_Pad1.33x1.80mm_HandSolder, F.Cu at (133.3, 69.2)
- added C5: 100u, Capacitor_SMD:C_1206_3216Metric_Pad1.33x1.80mm_HandSolder, F.Cu at (119.1, 68.3)
- added C6: 10u, Capacitor_SMD:C_1206_3216Metric_Pad1.33x1.80mm_HandSolder, F.Cu at (132.3, 81.6)
- added C7: 10u, Capacitor_SMD:C_1206_3216Metric_Pad1.33x1.80mm_HandSolder, F.Cu at (134.8, 81.6)
- added C8: 1u, Capacitor_SMD:C_1206_3216Metric_Pad1.33x1.80mm_HandSolder, F.Cu at (134.8, 87.7)
- added C9: 1u, Capacitor_SMD:C_1206_3216Metric_Pad1.33x1.80mm_HandSolder, F.Cu at (135.3, 98.1)
- added D1: D_Schottky, Diode_SMD:D_PowerDI-123, F.Cu at (128.5, 80.0)
- added D2: D_Schottky, Diode_SMD:D_MicroSMP_AK, F.Cu at (135.2, 100.2)
- added JP1: Jumper_2_Bridged, Connector_PinHeader_2.54mm:PinHeader_1x02_P2.54mm_Vertical, F.Cu at (134.8, 63.9)
- added L1: 2.2uH, ul_LQH5BPN2R2N38L:IND_LQH5BPN_MUR, F.Cu at (127.0, 75.0)
- added R1: 100k, Resistor_SMD:R_1206_3216Metric_Pad1.30x1.75mm_HandSolder, F.Cu at (116.9, 85.8)
- added R10: 200k, Resistor_SMD:R_1206_3216Metric_Pad1.30x1.75mm_HandSolder, F.Cu at (138.5, 78.6)
- added R11: 22k, Resistor_SMD:R_1206_3216Metric_Pad1.30x1.75mm_HandSolder, F.Cu at (138.5, 73.6)
- added R2: 18k, Resistor_SMD:R_1206_3216Metric_Pad1.30x1.75mm_HandSolder, F.Cu at (111.8, 85.8)
- added R3: 47k, Resistor_SMD:R_1206_3216Metric_Pad1.30x1.75mm_HandSolder, F.Cu at (109.3, 71.5)
- added R4: 25m, Resistor_SMD:R_1206_3216Metric_Pad1.30x1.75mm_HandSolder, F.Cu at (123.5, 69.9)
- added R5: 0, Resistor_SMD:R_1206_3216Metric_Pad1.30x1.75mm_HandSolder, F.Cu at (118.9, 77.3)
- added R6: 10k, Resistor_SMD:R_1206_3216Metric_Pad1.30x1.75mm_HandSolder, F.Cu at (113.7, 67.3)
- added R7: 470, Resistor_SMD:R_1206_3216Metric_Pad1.30x1.75mm_HandSolder, F.Cu at (109.3, 68.2)
- added R8: 0, Resistor_SMD:R_1206_3216Metric_Pad1.30x1.75mm_HandSolder, F.Cu at (133.3, 66.8)
- added R9: 1M, Resistor_SMD:R_1206_3216Metric_Pad1.30x1.75mm_HandSolder, F.Cu at (134.8, 71.6)
- added TP1: TestPoint, Connector_PinHeader_2.54mm:PinHeader_1x01_P2.54mm_Vertical, F.Cu at (137.9, 83.1)
- added TP2: TestPoint, Connector_PinHeader_2.54mm:PinHeader_1x01_P2.54mm_Vertical, F.Cu at (107.5, 86.3)
- added U1: BD50HC0WEFJ, HTSOP-J8:HTSOP-J8, F.Cu at (138.3, 92.8)
- added U2: SY21222ABC, Package_TO_SOT_SMD:SOT-23-6, F.Cu at (131.9, 75.0)
- added U3: LTC2943, Package_DFN_QFN:DFN-8-1EP_3x3mm_P0.5mm_EP1.66x2.38mm, F.Cu at (123.6, 66.9)
- added U4: TPS259620DDAR, TPS25963x:SOIC-8-1EP_3.9x5.75mm_P1.27mm_EP2.4x3.1mm, F.Cu at (113.1, 77.4)
Routing:
- net +5V: track 0.00 -> 47.1 mm, vias 0 -> 2
- net Net-(U4-OVCSEL): track 0.00 -> 20.7 mm, vias 0 -> 2
- net GND: track 0.00 -> 16.4 mm, vias 0 -> 59
- net Net-(JP1-A): track 0.00 -> 11.4 mm
- net Net-(U4-EN/UVLO): track 0.00 -> 7.66 mm
- net Net-(U4-ILM): track 0.00 -> 7.56 mm
- net FAULT: track 0.00 -> 7.49 mm, vias 0 -> 1
- net Net-(U4-dVdt): track 0.00 -> 3.12 mm
- net +6V: track 0.00 -> 2.51 mm
- net VPACK: track 0.00 -> 2.35 mm
- net ALERT: track 0.00 -> 2.31 mm, vias 0 -> 1
- net Net-(JP1-B): track 0.00 -> 2.28 mm
- net SDA: track 0.00 -> 1.33 mm, vias 0 -> 1
- net SCL: track 0.00 -> 1.33 mm, vias 0 -> 1
- added copper zone on F.Cu, net +6V
- added copper zone on F.Cu, net +BATT
- added copper zone on B.Cu, net GND
- added copper zone on F.Cu, net GND
- added copper zone on F.Cu, net Net-(D1-A)
- added copper zone on F.Cu, net Net-(D2-A)
- added copper zone on F.Cu, net Net-(JP1-B)
- added copper zone on F.Cu, net Net-(U2-FB)
- added copper zone on F.Cu, net VPACK
Other:
- board text removed: "LPI2C0_SCL"
- board text removed: "LPI2C0_SDA"

Commit message: add memory module and increase size of shield
Parts:
- added J7: Conn_01x08_Socket, Connector_PinSocket_2.54mm:PinSocket_1x08_P2.54mm_Vertical, F.Cu at (137.0, 63.5)
- added J8: Conn_01x08_Socket, Connector_PinSocket_2.54mm:PinSocket_1x08_P2.54mm_Vertical, F.Cu at (136.9, 86.4)
- added R12: 10k, Resistor_SMD:R_1206_3216Metric_Pad1.30x1.75mm_HandSolder, F.Cu at (150.9, 82.9)
- moved D2 28.0 mm to (132.9, 128.1)
- moved BT1 28.0 mm to (117.4, 125.9)
- moved BT2 28.0 mm to (117.4, 121.3)
- moved C1 28.0 mm to (114.6, 116.2)
- moved C2 28.0 mm to (108.5, 111.2)
- moved C3 28.0 mm to (124.9, 96.4)
- moved C4 28.0 mm to (131.1, 97.0)
- moved C5 28.0 mm to (116.8, 96.2)
- moved C6 28.0 mm to (130.0, 109.4)
- moved C7 28.0 mm to (132.5, 109.4)
- moved C8 28.0 mm to (132.6, 115.5)
- moved C9 28.0 mm to (133.1, 125.9)
- moved D1 28.0 mm to (126.2, 107.8)
- moved H1 28.0 mm to (102.4, 140.3)
- moved H2 28.0 mm to (102.4, 89.9)
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Connections:
- J3 pad 9: 5V0_OUT -> +5V
- J5 pad 2: 5V0_OUT -> +5V
- U3 pad 4: SCL -> /P1_9
- U3 pad 5: SDA -> /P1_8
Routing:
- net +5V: track 47.1 -> 81.2 mm
- net /P2_6: track 0.00 -> 31.0 mm
- net /P1_8: track 0.00 -> 23.6 mm, vias 0 -> 1
- net /P1_9: track 0.00 -> 17.6 mm, vias 0 -> 1
- net /P2_16: track 0.00 -> 10.5 mm
- net /P2_13: track 0.00 -> 6.06 mm
- net /P2_12: track 0.00 -> 6.06 mm
- net +3V3: track 0.00 -> 4.44 mm
- net SDA: track 1.33 -> 0.00 mm, vias 1 -> 0
- net SCL: track 1.33 -> 0.00 mm, vias 1 -> 0
Other:
- board size 101.4 x 54.6 mm -> 101.5 x 82.1 mm
