File: FRDM-MCXA153_shield_template.kicad_sch (KiCad schematic)
At the start: 6 parts, among them J1 Conn_02x08_Odd_Even, J2 Conn_02x10_Odd_Even, J3 Conn_02x08_Odd_Even, J4 Conn_02x06_Odd_Even, J5 Conn_01x08_Pin, J6 Conn_01x08_Pin

Commit message: add power module
Other:
- added sheet PowerModule (PowerModule.kicad_sch)
- company: Alessandro Lo Monaco -> HANdeld Horizons
- moved on the sheet: J1, J2, J3, J4, J5, J6

Commit message: add memory module and increase size of shield
Connections:
- net 5V0_OUT renamed +5V
Other:
- added sheet MemoryModule (MemoryModule.kicad_sch)
- sheet PowerModule ports: added SCL, SDA; removed none
