File: PowerModule.kicad_sch (KiCad schematic)
At the start: 32 parts, among them U1 BD50HC0WEFJ, U2 SY21222ABC, U3 LTC2943, U4 TPS259620DDAR

Commit message: add memory module and increase size of shield
Changed lines of the file:
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@@
 		)
 	)
-	(global_label "SCL"
+	(hierarchical_label "SCL"
 		(shape input)
 		(at 36.83 53.34 180)
-		(fields_autoplaced yes)
 		(effects
 			(font
@@
 			(justify right)
 		)
-		(property "Intersheetrefs" "${INTERSHEET_REFS}"
-			(at 30.3372 53.34 0)
-			(effects
-				(font
-					(size 1.27 1.27)
-				)
-				(justify right)
-				(hide yes)
-			)
-		)
 	)
-	(global_label "SDA"
+	(hierarchical_label "SDA"
 		(shape input)
 		(at 36.83 50.8 180)
-		(fields_autoplaced yes)
 		(effects
 			(font
@@
 			(justify right)
 		)
-		(property "Intersheetrefs" "${INTERSHEET_REFS}"
-			(at 30.2767 50.8 0)
-			(effects
-				(font
-					(size 1.27 1.27)
-				)
-				(justify right)
-				(hide yes)
-			)
-		)
 	)
